Commit message: final software review

File: modelos/3dof.urdf (robot description, URDF)
Before this commit: robot threeseg, 5 links, 4 joints
Links:
- link link_1: geometry visual box size=0.1 0.4 1

File: modelos/cartesian.urdf (robot description, URDF)
Before this commit: robot CartMan, 13 links, 12 joints
Links:
- removed link link_support1
- removed link link_support1x
- removed link link_support1y
- removed link link_support2
- removed link link_support2x
- removed link link_support2y
- removed link link_support3
- removed link link_support4
- added link link_supportz; visual box size=0.07 0.07 1; visual box size=0.07 0.07 1
Joints:
- removed joint base_support1x
- removed joint base_support1y
- removed joint base_support2
- removed joint base_support2x
- removed joint base_support2y
- removed joint base_support3
- removed joint base_support4
- joint base_support1: child link_support1 -> link_supportz; origin xyz=0 0 -0.5 rpy=0 0 0 -> xyz=0 0 0 rpy=0 0 0
- joint joint_3: origin xyz=0 0.12 0 rpy=0 0 0 -> xyz=0 -0.55 0 rpy=0 0 0

File: modelos/cylindrical.urdf (robot description, URDF)
Before this commit: robot Cylindrical, 5 links, 4 joints
Joints:
- joint joint_2: limit lower=0 upper=0.85 effort=1000.0 velocity=1.0 -> lower=0 upper=0.82 effort=1000.0 velocity=1.0

Commit message: LVR Final

File: modelos/3dof.urdf (robot description, URDF)
Before this commit: robot threeseg, 5 links, 4 joints
Links:
- link link_1: geometry visual box size=0.2 0.2 1
- link link_3: geometry visual box size=0.2 0.2 0.5

File: modelos/3dofPrueba.urdf (robot description, URDF)
Before this commit: robot 3dof, 4 links, 3 joints
Links:
- added link link_3; visual box size=0.1 0.1 1.0
- link link_1: geometry visual box size=0.3 0.3 1.5
Joints:
- removed joint joint_2-tool0
- added joint joint_3: type revolute, parent link_2, child link_3, origin xyz=0 0 1 rpy=0 0 0, axis 0 1 0, limit lower=-3.14 upper=3.14 effort=30 velocity=1.0
- added joint joint_3-tool0: type revolute, parent link_3, child tool0, origin xyz=0 0 1.0 rpy=0 0 0, axis 0 0 1, limit lower=-6.28318 upper=6.28318 effort=30 velocity=1.0

File: modelos/3dofUNI.urdf (robot description, URDF)
Before this commit: robot 3dof, 4 links, 3 joints
Links:
- added link link_3; visual box size=0.1 0.1 1.0
- link link_1: geometry visual box size=0.3 0.3 1.5
Joints:
- removed joint joint_2-tool0
- added joint joint_3: type revolute, parent link_2, child link_3, origin xyz=0 0 1 rpy=0 0 0, axis 0 1 0, limit lower=-3.14 upper=3.14 effort=30 velocity=1.0
- added joint joint_3-tool0: type revolute, parent link_3, child tool0, origin xyz=0 0 1.0 rpy=0 0 0, axis 0 0 1, limit lower=-6.28318 upper=6.28318 effort=30 velocity=1.0
- joint joint_1: limit lower=-3.14 upper=3.14 effort=30 velocity=1.0 -> lower=-3.14 upper=0 effort=30 velocity=1.0

File: modelos/cylindrical.urdf (robot description, URDF)
Before this commit: robot Cylindrical, 5 links, 4 joints
Links:
- link link_1: geometry visual cylinder length=1.0 radius=0.09
